File: hardware/tonberry-pico/tonberry-pico.kicad_pcb (KiCad board)
At the start: 2 copper layers, 98 x 53.5 mm, 32 parts, among them J1 MicroSD_Breakout, J2 SparkFun I2S Audio Breakout M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, J3 RC522_Breakout, J4 Adafruit_bq25185_5V, J5 UART, J6 WS2812, J7 Buttons, J8 Conn_01x01, J9 MSD-6-A, Q1 2N7000, Q2 2N7000, SW5 SW_Push, U1 RaspberryPi_Pico_W

Commit message: as per request in the PR, I adjusted the following items: - applied same track width (0.4064) - removed the SD_CD line
Routing:
- net /SD_CD: track 29.1 -> 0.00 mm
- net /SD_CS: track 32.9 -> 32.2 mm
Changed lines of the file:
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@@
 	)
 	(segment
-		(start 137.7056 48.0056)
-		(end 143.8906 48.0056)
-		(width 0.2032)
+		(start 138.104 47.904)
+		(end 143.789 47.904)
+		(width 0.4064)
+		(layer "F.Cu")
+		(net "/SD_SCK")
+	)
+	(segment
+		(start 136.2 44.6)
+		(end 136.2 46)
+		(width 0.4064)
+		(layer "F.Cu")
+		(net "/SD_SCK")
+	)
+	(segment
+		(start 136.2 46)
+		(end 138.104 47.904)
+		(width 0.4064)
+		(layer "F.Cu")
+		(net "/SD_SCK")
+	)
+	(segment
+		(start 143.789 47.904)
+		(end 144.78 48.895)
+		(width 0.4064)
 		(layer "F.Cu")
 		(net "/SD_SCK")
@@
 	)
 	(segment
-		(start 136.2 44.6)
-		(end 136.2 46.5)
-		(width 0.2032)
-		(layer "F.Cu")
-		(net "/SD_SCK")
-	)
-	(segment
-		(start 143.8906 48.0056)
-		(end 144.78 48.895)
-		(width 0.2032)
-		(layer "F.Cu")
-		(net "/SD_SCK")
-	)
-	(segment
-		(start 136.2 46.5)
-		(end 137.7056 48.0056)
-		(width 0.2032)
-		(layer "F.Cu")
-		(net "/SD_SCK")
+		(start 134 44.6)
+		(end 134 46.8)
+		(width 0.4064)
+		(layer "F.Cu")
+		(net "/SD_DI")
+	)
+	(segment
+		(start 134 46.8)
+		(end 139.592835 52.392835)
+		(width 0.4064)
+		(layer "F.Cu")
+		(net "/SD_DI")
 	)
 	(segment
@@
 	)
 	(segment
-		(start 142.8944 52.0894)
-		(end 144.78 53.975)
-		(width 0.2032)
-		(layer "F.Cu")
-		(net "/SD_DI")
-	)
-	(segment
-		(start 139.2894 52.0894)
-		(end 142.8944 52.0894)
-		(width 0.2032)
-		(layer "F.Cu")
-		(net "/SD_DI")
-	)
-	(segment
-		(start 134 44.6)
-		(end 134 46.8)
-		(width 0.2032)
-		(layer "F.Cu")
-		(net "/SD_DI")
-	)
-	(segment
 		(start 158.75 51.435)
 		(end 157.48 52.705)
@@
 	)
 	(segment
+		(start 139.592835 52.392835)
+		(end 143.197835 52.392835)
+		(width 0.4064)
+		(layer "F.Cu")
+		(net "/SD_DI")
+	)
+	(segment
 		(start 145.415 53.975)
 		(end 144.78 53.975)
@@
 	)
 	(segment
-		(start 134 46.8)
-		(end 139.2894 52.0894)
-		(width 0.2032)
+		(start 143.197835 52.392835)
+		(end 144.78 53.975)
+		(width 0.4064)
 		(layer "F.Cu")
 		(net "/SD_DI")
@@
 		(start 146.065 45.1)
 		(end 144.78 43.815)
-		(width 0.2032)
+		(width 0.4064)
 		(layer "F.Cu")
 		(net "/SD_DO")
@@
 		(start 151.175 53.975)
 		(end 150.8 53.6)
-		(width 0.2032)
+		(width 0.4064)
 		(layer "F.Cu")
 		(net "/SD_DO")
 	)
 	(segment
-		(start 142.9656 45.6294)
+		(start 142.776 45.819)
 		(end 144.78 43.815)
-		(width 0.2032)
-		(layer "F.Cu")
-		(net "/SD_DO")
-	)
-	(segment
-		(start 138.4 45.2088)
-		(end 138.8206 45.6294)
-		(width 0.2032)
+		(width 0.4064)
 		(layer "F.Cu")
 		(net "/SD_DO")
@@
 		(start 150.3 45.1)
 		(end 146.065 45.1)
-		(width 0.2032)
+		(width 0.4064)
 		(layer "F.Cu")
 		(net "/SD_DO")
 	)
 	(segment
+		(start 138.8 45.819)
+		(end 142.776 45.819)
+		(width 0.4064)
+		(layer "F.Cu")
+		(net "/SD_DO")
+	)
+	(segment
 		(start 138.4 44.6)
-		(end 138.4 45.2088)
-		(width 0.2032)
+		(end 138.4 45.419)
+		(width 0.4064)
+		(layer "F.Cu")
+		(net "/SD_DO")
+	)
+	(segment
+		(start 138.4 45.419)
+		(end 138.8 45.819)
+		(width 0.4064)
 		(layer "F.Cu")
 		(net "/SD_DO")
@@
 		(start 158.75 53.975)
 		(end 151.175 53.975)
-		(width 0.2032)
-		(layer "F.Cu")
-		(net "/SD_DO")
-	)
-	(segment
-		(start 138.8206 45.6294)
-		(end 142.9656 45.6294)
-		(width 0.2032)
+		(width 0.4064)
 		(layer "F.Cu")
 		(net "/SD_DO")
@@
 		(start 150.8 53.6)
 		(end 150.8 45.6)
-		(width 0.2032)
+		(width 0.4064)
 		(layer "B.Cu")
 		(net "/SD_DO")
@@
 		(start 150.8 45.6)
 		(end 150.3 45.1)
-		(width 0.2032)
+		(width 0.4064)
 		(layer "B.Cu")
 		(net "/SD_DO")
 	)
 	(segment
-		(start 132.9 46.7)
-		(end 138.8 52.6)
-		(width 0.2032)
+		(start 132.9 44.8)
+		(end 132.9 47.2)
+		(width 0.4064)
 		(layer "F.Cu")
 		(net "/SD_CS")
 	)
 	(segment
-		(start 143.3 53.1)
-		(end 143.3 55.035)
-		(width 0.2032)
+		(start 138.989725 53.289725)
+		(end 139.989725 53.289725)
+		(width 0.4064)
 		(layer "F.Cu")
 		(net "/SD_CS")
 	)
 	(segment
-		(start 132.9 44.8)
-		(end 132.9 46.7)
-		(width 0.2032)
+		(start 144.695 56.6)
+		(end 144.78 56.515)
+		(width 0.4064)
 		(layer "F.Cu")
 		(net "/SD_CS")
 	)
 	(segment
-		(start 138.8 52.6)
-		(end 142.8 52.6)
-		(width 0.2032)
+		(start 143.3 56.6)
+		(end 144.695 56.6)
+		(width 0.4064)
 		(layer "F.Cu")
 		(net "/SD_CS")
 	)
 	(segment
-		(start 143.3 55.035)
-		(end 144.78 56.515)
-		(width 0.2032)
+		(start 132.9 47.2)
+		(end 138.989725 53.289725)
+		(width 0.4064)
 		(layer "F.Cu")
 		(net "/SD_CS")
 	)
 	(segment
-		(start 142.8 52.6)
-		(end 143.3 53.1)
-		(width 0.2032)
+		(start 139.989725 53.289725)
+		(end 143.3 56.6)
+		(width 0.4064)
 		(layer "F.Cu")
 		(net "/SD_CS")
@@
 	)
 	(segment
+		(start 135.1 46.4)
+		(end 140.135 51.435)
+		(width 0.4064)
+		(layer "F.Cu")
+		(net "+3V3")
+	)
+	(segment
 		(start 144.78 51.435)
 		(end 148.67 51.435)
@@
 	)
 	(segment
-		(start 139.635 51.435)
-		(end 141.135 51.435)
-		(width 0.4064)
-		(layer "F.Cu")
-		(net "+3V3")
-	)
-	(segment
 		(start 150.495 51.475)
 		(end 151.79 50.18)
@@
 	)
 	(segment
-		(start 135.1 44.4)
-		(end 135.1 46.9)
-		(width 0.4064)
-		(layer "F.Cu")
-		(net "+3V3")
-	)
-	(segment
 		(start 159.440958 50.18)
 		(end 159.425958 50.165)
@@
 	)
 	(segment
+		(start 135.1 44.4)
+		(end 135.1 46.4)
+		(width 0.4064)
+		(layer "F.Cu")
+		(net "+3V3")
+	)
+	(segment
 		(start 139.065 74.295)
 		(end 139.065 66.085)
@@
 	)
 	(segment
-		(start 135.1 46.9)
-		(end 139.635 51.435)
-		(width 0.4064)
-		(layer "F.Cu")
-		(net "+3V3")
-	)
-	(segment
 		(start 170.195 57.77)
 		(end 176.53 51.435)
@@
 	)
 	(segment
-		(start 144.78 51.435)
-		(end 141.135 51.435)
+		(start 140.135 51.435)
+		(end 144.78 51.435)
 		(width 0.4064)
 		(layer "F.Cu")
@@
 	)
 	(segment
-		(start 138.7 53.9968)
-		(end 138.7 54.9)
-		(width 0.2032)
-		(layer "F.Cu")
-		(net "/SD_CD")
-	)
-	(segment
-		(start 142.9838 41.275)
-		(end 140.9794 43.2794)
-		(width 0.2032)
-		(layer "F.Cu")
-		(net "/SD_CD")
-	)
-	(segment
-		(start 131.1206 43.5706)
-		(end 131.1206 46.4174)
-		(width 0.2032)
-		(layer "F.Cu")
-		(net "/SD_CD")
-	)
-	(segment
-		(start 131.4118 43.2794)
-		(end 131.1206 43.5706)
-		(width 0.2032)
-		(layer "F.Cu")
-		(net "/SD_CD")
-	)
-	(segment
-		(start 131.1206 46.4174)
-		(end 138.7 53.9968)
-		(width 0.2032)
-		(layer "F.Cu")
-		(net "/SD_CD")
-	)
-	(segment
-		(start 140.9794 43.2794)
-		(end 131.4118 43.2794)
-		(width 0.2032)
-		(layer "F.Cu")
-		(net "/SD_CD")
-	)
-	(segment
-		(start 144.78 41.275)
-		(end 142.9838 41.275)
-		(width 0.2032)
-		(layer "F.Cu")
-		(net "/SD_CD")
-	)
-	(segment
